File: electrical/banana17_main/banana17_matrix.kicad_sch (KiCad schematic)
At the start: 38 parts, among them SW1 SW, SW10 SW, SW11 SW, SW12 SW, SW13 SW, SW14 SW, SW15 SW, SW16 SW, SW17 SW, SW2 SW, SW3 SW, SW4 SW, SW5 SW, SW6 SW, SW7 SW, SW8 SW, SW9 SW

Commit message: RP2040 routed.
RP2040 routed.
Connections:
- net ROW3: no longer D15.1 (K)
- net ROW4: now also D15.1 (K)
Other:
- moved on the sheet: D15, SW15
Changed lines of the file:
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@@
 	)
 	(junction
-		(at 175.26 92.71)
+		(at 114.3 82.55)
 		(diameter 0)
 		(color 0 0 0 0)
 	)
 	(junction
-		(at 114.3 82.55)
+		(at 137.16 168.91)
 		(diameter 0)
 		(color 0 0 0 0)
@@
 	)
 	(junction
+		(at 175.26 92.71)
+		(diameter 0)
+		(color 0 0 0 0)
+	)
+	(junction
 		(at 137.16 82.55)
 		(diameter 0)
@@
 	)
 	(junction
-		(at 137.16 147.32)
-		(diameter 0)
-		(color 0 0 0 0)
-	)
-	(junction
 		(at 91.44 104.14)
 		(diameter 0)
@@
 	(wire
 		(pts
-			(xy 160.02 138.43) (xy 160.02 135.89)
+			(xy 158.75 160.02) (xy 158.75 157.48)
 		)
 		(stroke
@@
 	(wire
 		(pts
-			(xy 160.02 135.89) (xy 161.29 135.89)
+			(xy 158.75 157.48) (xy 160.02 157.48)
 		)
 		(stroke
@@
 	(wire
 		(pts
-			(xy 137.16 147.32) (xy 160.02 147.32)
-		)
-		(stroke
-			(width 0)
-			(type default)
-		)
-	)
-	(wire
-		(pts
 			(xy 137.16 102.87) (xy 137.16 104.14)
 		)
@@
 	(wire
 		(pts
-			(xy 171.45 135.89) (xy 175.26 135.89)
+			(xy 170.18 157.48) (xy 175.26 157.48)
 		)
 		(stroke
@@
 	(wire
 		(pts
+			(xy 137.16 168.91) (xy 158.75 168.91)
+		)
+		(stroke
+			(width 0)
+			(type default)
+		)
+	)
+	(wire
+		(pts
 			(xy 59.69 111.76) (xy 59.69 133.35)
 		)
@@
 	(wire
 		(pts
-			(xy 175.26 92.71) (xy 175.26 135.89)
+			(xy 175.26 92.71) (xy 175.26 157.48)
 		)
 		(stroke
@@
 	(wire
 		(pts
-			(xy 160.02 146.05) (xy 160.02 147.32)
+			(xy 158.75 167.64) (xy 158.75 168.91)
 		)
 		(stroke
@@
 	(symbol
 		(lib_id "Switch:SW_SPST")
-		(at 166.37 135.89 0)
+		(at 165.1 157.48 0)
 		(unit 1)
 		(exclude_from_sim no)
@@
 		(fields_autoplaced yes)
 		(property "Reference" "SW15"
-			(at 166.37 129.54 0)
+			(at 165.1 151.13 0)
 			(effects
 				(font
@@
 		)
 		(property "Value" "SW"
-			(at 166.37 132.08 0)
+			(at 165.1 153.67 0)
 			(effects
 				(font
@@
 		)
 		(property "Footprint" "MX_Hotswap:MX-Hotswap-2U-Vertical"
-			(at 166.37 135.89 0)
+			(at 165.1 157.48 0)
 			(effects
 				(font
@@
 		)
 		(property "Datasheet" "~"
-			(at 166.37 135.89 0)
+			(at 165.1 157.48 0)
 			(effects
 				(font
@@
 		)
 		(property "Description" "Single Pole Single Throw (SPST) switch"
-			(at 166.37 135.89 0)
+			(at 165.1 157.48 0)
 			(effects
 				(font
@@
 	(symbol
 		(lib_id "Device:D")
-		(at 160.02 142.24 90)
+		(at 158.75 163.83 90)
 		(unit 1)
 		(exclude_from_sim no)
@@
 		(fields_autoplaced yes)
 		(property "Reference" "D15"
-			(at 162.56 140.9699 90)
+			(at 161.29 162.5599 90)
 			(effects
 				(font
@@
 		)
 		(property "Value" "D"
-			(at 162.56 143.5099 90)
+			(at 161.29 165.0999 90)
 			(effects
 				(font
@@
 		)
 		(property "Footprint" "Diode_SMD:D_0805_2012Metric_Pad1.15x1.40mm_HandSolder"
-			(at 160.02 142.24 0)
+			(at 158.75 163.83 0)
 			(effects
 				(font
@@
 		)
 		(property "Datasheet" "~"
-			(at 160.02 142.24 0)
+			(at 158.75 163.83 0)
 			(effects
 				(font
@@
 		)
 		(property "Description" "Diode"
-			(at 160.02 142.24 0)
+			(at 158.75 163.83 0)
 			(effects
 				(font
@@
 		)
 		(property "Sim.Device" "D"
-			(at 160.02 142.24 0)
+			(at 158.75 163.83 0)
 			(effects
 				(font
@@
 		)
 		(property "Sim.Pins" "1=K 2=A"
-			(at 160.02 142.24 0)
+			(at 158.75 163.83 0)
 			(effects
 				(font
